File: PRKL30.kicad_pcb (KiCad board)
At the start: 2 copper layers, 83 parts, among them K1 KEYSW, K10 KEYSW, K11 KEYSW, K12 KEYSW, K14 KEYSW, K15 KEYSW, K16 KEYSW, K17 KEYSW, K18 KEYSW, K19 KEYSW, K2 KEYSW, K20 KEYSW, K21 KEYSW, K22 KEYSW, K23 KEYSW, K24 KEYSW, K25 KEYSW, K27 KEYSW, K28 KEYSW, K29 KEYSW, K3 KEYSW, K30 KEYSW, K31 KEYSW, K32 KEYSW, K33 KEYSW, K34 KEYSW, K35 KEYSW, K36 KEYSW, K37 KEYSW, K4 KEYSW, K5 KEYSW, K6 KEYSW, K7 KEYSW, K8 KEYSW, K9 KEYSW

Commit message: Change project name, clean up older files
Parts:
- added Feather1: Adafruit32u4BLE, SpaceLib:Adafruit32u4BLE, F.Cu at (100.8, 77.6)
- added M3_1: VAL**, keyboard_parts:HOLE_M3, F.Cu at (71.4, 76.2)
- added M3_2: VAL**, keyboard_parts:HOLE_M3, F.Cu at (90.5, 107.2)
- added M3_3: VAL**, keyboard_parts:HOLE_M3, F.Cu at (128.5, 76.2)
- added M3_4: VAL**, keyboard_parts:HOLE_M3, F.Cu at (185.4, 76.2)
- added M3_5: VAL**, keyboard_parts:HOLE_M3, F.Cu at (204.8, 109.5)
- added M3_6: VAL**, keyboard_parts:HOLE_M3, F.Cu at (242.9, 76.0)
- added M3_7: VAL**, keyboard_parts:HOLE_M3, F.Cu at (296.5, 77.4)
- added SW2: SW_SPDT, Button_Switch_SMD:SW_SPDT_PCM12, B.Cu at (283.3, 58.0)
- LED_DATA1: value DATA -> 0
- LED_GND1: value GND -> 0
- LED_PWR1: value PWR -> 0
- MCU_Pro_Micr0: moved to B.Cu
- moved D16 28.9 mm to (119.9, 74.7)
- moved D32 22.9 mm to (148.9, 105.4), turned to 90 degrees
- moved D29 17.9 mm to (127.3, 104.6)
- moved D3 17.8 mm to (82.4, 75.3)
- moved D28 17.6 mm to (72.8, 104.3)
- moved D23 14.7 mm to (243.3, 85.2), turned to 90 degrees
- moved D13 14.3 mm to (283.5, 67.6), turned to 90 degrees
- moved D17 13.8 mm to (127.8, 85.1), turned to 90 degrees
- moved D24 13.6 mm to (260.9, 85.3), turned to 90 degrees
- moved D8 13.5 mm to (185.4, 66.5), turned to 90 degrees
- moved D18 13.2 mm to (147.5, 86.6), turned to 90 degrees
- moved D12 13.2 mm to (261.6, 66.5), turned to 90 degrees
- moved D7 13.2 mm to (166.6, 66.5), turned to 90 degrees
- moved D10 13.1 mm to (223.5, 66.5), turned to 90 degrees
- moved D11 13.1 mm to (242.8, 66.5), turned to 90 degrees
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Connections:
- MCU_Pro_Micr0 pad 21: RGB_PWR -> Net-(MCU_Pro_Micr0-Pad21)
- MCU_Pro_Micr0 pad 24: Net-(MCU_Pro_Micr0-Pad24) -> RGB_PWR
Routing:
- net ColF: track 0.00 -> 330.5 mm
- net GND: track 0.00 -> 299.2 mm, vias 0 -> 1
- net ColC: track 0.00 -> 287.9 mm
- net RowD: track 0.00 -> 275.4 mm
- net ColB: track 0.00 -> 273.0 mm
- net ColH: track 0.00 -> 268.6 mm, vias 0 -> 1
- net ColA: track 0.00 -> 267.3 mm
- net ColD: track 0.00 -> 255.2 mm
- net ColE: track 0.00 -> 253.9 mm, vias 0 -> 2
- net RowC: track 0.00 -> 244.5 mm
- net RowB: track 0.00 -> 241.8 mm, vias 0 -> 1
- net ColG: track 0.00 -> 238.5 mm
- net RowA: track 0.00 -> 215.9 mm
- net ColJ: track 0.00 -> 212.2 mm
- net DP1: track 0.00 -> 209.4 mm
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Other:
- board outline added: 254.9 x 62.2 mm
