File: PRKL30.kicad_pcb (KiCad board)
At the start: 2 copper layers, 254.9 x 63.5 mm, 94 parts, among them K1 KEYSW, K10 KEYSW, K11 KEYSW, K12 KEYSW, K14 KEYSW, K15 KEYSW, K16 KEYSW, K17 KEYSW, K18 KEYSW, K19 KEYSW, K2 KEYSW, K20 KEYSW, K21 KEYSW, K22 KEYSW, K23 KEYSW, K24 KEYSW, K25 KEYSW, K27 KEYSW, K28 KEYSW, K29 KEYSW, K3 KEYSW, K30 KEYSW, K31 KEYSW, K32 KEYSW, K33 KEYSW, K34 KEYSW, K35 KEYSW, K36 KEYSW, K37 KEYSW, K4 KEYSW, K5 KEYSW, K6 KEYSW, K7 KEYSW, K8 KEYSW, K9 KEYSW, M2_1 VAL**, M2_2 VAL**, M2_3 VAL**, M2_4 VAL**, M2_5 VAL**, M2_6 VAL**, M2_7 VAL**, SW2 SW_SPDT

Commit message: moved ble switch and edited pcb outlines and traces related to that
Parts:
- moved SW2 3.05 mm to (283.3, 55.9)
Routing:
- net GND: track 308.7 -> 310.1 mm
Other:
- board size 254.9 x 63.5 mm -> 254.9 x 62.2 mm
Changed lines of the file:
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@@
-(kicad_pcb (version 20171130) (host pcbnew "(5.0.1)-3")
+(kicad_pcb (version 20171130) (host pcbnew "(5.1.5)-3")
   (general
     (thickness 1.6)
-    (drawings 24)
-    (tracks 1287)
+    (drawings 22)
+    (tracks 1292)
     (zones 0)
     (modules 94)
@@
     (zone_45_only no)
     (trace_min 0.2)
-    (segment_width 0.2)
-    (edge_width 0.15)
     (via_size 0.8)
     (via_drill 0.4)
@@
     (uvia_min_size 0.2)
     (uvia_min_drill 0.1)
+    (edge_width 0.15)
+    (segment_width 0.2)
     (pcb_text_width 0.3)
     (pcb_text_size 1.5 1.5)
@@
   )
   (module Button_Switch_SMD:SW_SPDT_PCM12 (layer B.Cu)
-    (at 283.3 52.8946)
+    (at 283.3 55.9426)
     (descr "Ultraminiature Surface Mount Slide Switch, right-angle, https://www.ckswitches.com/media/1424/pcm.pdf")
     (attr smd)
@@
     )
   )
-  (gr_line (start 278.846 52.036) (end 278.846 57.126) (layer Edge.Cuts) (width 0.2))
-  (gr_line (start 287.756 52.046) (end 287.756 57.126) (layer Edge.Cuts) (width 0.2))
   (gr_arc (start 87.74 56.15) (end 87.74 57.15) (angle -90) (layer Edge.Cuts) (width 0.15))
   (gr_arc (start 53.38 58.14) (end 53.38 57.14) (angle -90) (layer Edge.Cuts) (width 0.15))
-  (gr_line (start 279.05 50.7846) (end 287.55 50.7846) (layer Edge.Cuts) (width 0.15))
-  (gr_line (start 287.75 52.0446) (end 287.75 50.9846) (layer Edge.Cuts) (width 0.15))
-  (gr_line (start 278.85 52.0446) (end 278.85025 50.994588) (layer Edge.Cuts) (width 0.15))
-  (gr_arc (start 279.05 50.9846) (end 279.05 50.7846) (angle -92.86240523) (layer Edge.Cuts) (width 0.15))
-  (gr_arc (start 287.55 50.9846) (end 287.75 50.9846) (angle -90) (layer Edge.Cuts) (width 0.15))
+  (gr_line (start 279.05 53.8326) (end 287.55 53.8326) (layer Edge.Cuts) (width 0.15))
+  (gr_line (start 287.75 57.15) (end 287.75 54.0326) (layer Edge.Cuts) (width 0.15))
+  (gr_line (start 278.85 57.15) (end 278.85025 54.042588) (layer Edge.Cuts) (width 0.15))
+  (gr_arc (start 279.05 54.0326) (end 279.05 53.8326) (angle -92.86240523) (layer Edge.Cuts) (width 0.15))
+  (gr_arc (start 287.55 54.0326) (end 287.75 54.0326) (angle -90) (layer Edge.Cuts) (width 0.15))
   (gr_line (start 306.23 114.3) (end 53.37 114.29995) (layer Edge.Cuts) (width 0.15))
   (gr_line (start 52.38 113.3) (end 52.38 58.14) (layer Edge.Cuts) (width 0.15))
@@
   (segment (start 107.62 58.97) (end 108.1188 58.4712) (width 0.25) (layer F.Cu) (net 54))
   (segment (start 108.1188 58.4712) (end 254.1884 58.4712) (width 0.25) (layer F.Cu) (net 54))
-  (segment (start 277.8505 58.7509) (end 254.4681 58.7509) (width 0.25) (layer B.Cu) (net 54))
   (segment (start 254.4681 58.7509) (end 254.1884 58.4712) (width 0.25) (layer B.Cu) (net 54))
-  (segment (start 284.05 55.3999) (end 280.699 58.7509) (width 0.25) (layer B.Cu) (net 54))
-  (segment (start 280.699 58.7509) (end 277.8505 58.7509) (width 0.25) (layer B.Cu) (net 54))
-  (segment (start 277.8505 58.7509) (end 277.8505 63.5666) (width 0.25) (layer B.Cu) (net 54))
-  (segment (start 277.8505 63.5666) (end 266.1993 75.2178) (width 0.25) (layer B.Cu) (net 54))
-  (segment (start 266.1993 75.2178) (end 266.1993 78.1) (width 0.25) (layer B.Cu) (net 54))
   (segment (start 107.62 58.97) (end 94.3328 58.97) (width 0.25) (layer B.Cu) (net 54))
   (segment (start 94.3328 58.97) (end 93.1311 60.1717) (width 0.25) (layer B.Cu) (net 54))
@@
   (segment (start 91.1783 61.0123) (end 91.1783 64.9047) (width 0.25) (layer B.Cu) (net 54))
   (segment (start 91.1783 64.9047) (end 90.043 66.04) (width 0.25) (layer B.Cu) (net 54))
-  (segment (start 284.05 54.3246) (end 284.05 55.3999) (width 0.25) (layer B.Cu) (net 54))
   (segment (start 265.024 78.1) (end 258.724 78.1) (width 0.25) (layer B.Cu) (net 54))
   (segment (start 265.024 78.1) (end 266.1993 78.1) (width 0.25) (layer B.Cu) (net 54))
@@
   (segment (start 75.4748 87.0096) (end 65.5789 87.0096) (width 0.25) (layer B.Cu) (net 54))
   (via (at 254.1884 58.4712) (size 0.8) (layers F.Cu B.Cu) (net 54))
+  (segment (start 269.372 78.1) (end 266.1993 78.1) (width 0.25) (layer B.Cu) (net 54))
+  (segment (start 280.924 66.548) (end 269.372 78.1) (width 0.25) (layer B.Cu) (net 54))
+  (segment (start 284.05 57.3726) (end 284.05 58.596) (width 0.25) (layer B.Cu) (net 54))
+  (segment (start 280.924 61.722) (end 280.924 66.548) (width 0.25) (layer B.Cu) (net 54))
+  (segment (start 284.05 58.596) (end 280.924 61.722) (width 0.25) (layer B.Cu) (net 54))
+  (segment (start 280.924 61.722) (end 279.654 61.722) (width 0.25) (layer B.Cu) (net 54))
+  (segment (start 275.9209 58.7509) (end 276.6829 58.7509) (width 0.25) (layer B.Cu) (net 54))
+  (segment (start 275.9209 58.7509) (end 254.4681 58.7509) (width 0.25) (layer B.Cu) (net 54))
+  (segment (start 276.6829 58.7509) (end 279.654 61.722) (width 0.25) (layer B.Cu) (net 54))
   (segment (start 90.043 70.0203) (end 89.8326 69.8099) (width 0.25) (layer F.Cu) (net 55))
   (segment (start 89.8326 69.8099) (end 69.2873 69.8099) (width 0.25) (layer F.Cu) (net 55))
@@
   (segment (start 111.555 72.468) (end 110.363 73.66) (width 0.25) (layer B.Cu) (net 61))
   (via (at 111.4863 62.9278) (size 0.8) (layers F.Cu B.Cu) (net 61))
-  (segment (start 281.05 54.3246) (end 281.05 55.4098) (width 0.25) (layer B.Cu) (net 63))
-  (segment (start 281.05 55.4098) (end 278.8903 57.5695) (width 0.25) (layer B.Cu) (net 63))
-  (segment (start 278.8903 57.5695) (end 253.6308 57.5695) (width 0.25) (layer B.Cu) (net 63))
+  (segment (start 281.05 57.3726) (end 281.05 58.4578) (width 0.25) (layer B.Cu) (net 63))
   (segment (start 253.6308 57.5695) (end 250.6879 60.5124) (width 0.25) (layer B.Cu) (net 63))
   (segment (start 250.6879 60.5124) (end 247.3178 60.5124) (width 0.25) (layer F.Cu) (net 63))
@@
   (segment (start 112.1947 71.12) (end 110.363 71.12) (width 0.25) (layer F.Cu) (net 63))
   (via (at 250.6879 60.5124) (size 0.8) (layers F.Cu B.Cu) (net 63))
+  (segment (start 276.7715 57.5695) (end 277.5335 57.5695) (width 0.25) (layer B.Cu) (net 63))
+  (segment (start 276.7715 57.5695) (end 253.6308 57.5695) (width 0.25) (layer B.Cu) (net 63))
+  (segment (start 277.5335 57.5695) (end 279.146 59.182) (width 0.25) (layer B.Cu) (net 63))
+  (segment (start 280.3258 59.182) (end 281.05 58.4578) (width 0.25) (layer B.Cu) (net 63))
+  (segment (start 279.146 59.182) (end 280.3258 59.182) (width 0.25) (layer B.Cu) (net 63))
 )

Commit message: Push rev 1.1 with bigger mount holes to allow for M2 spacers
Parts:
- removed G_PB: LOGO_PB, MEEMIKEEBSILK:Pb
- LED_DATA1: value LED_DATA -> DATA
- LED_GND1: value LED_GND -> GND
- LED_PWR1: value LED_PWR -> +5V
- M2_1, M2_2, M2_3, M2_4, M2_5, M2_6, M2_7: footprint MountingHole:MountingHole_2.2mm_M2 -> kbd:spacer_m2
Routing:
- net ColE: track 243.9 -> 245.6 mm
- net RowD: track 315.8 -> 317.1 mm
- net ColF: track 289.9 -> 290.9 mm
- net ColD: track 206.1 -> 207.0 mm
- net ColA: track 263.7 -> 264.5 mm
- net DP1: track 179.9 -> 180.7 mm
- net RGB: track 62.2 -> 62.8 mm
