File: PRKL30.kicad_pcb (KiCad board)
At the start: 2 copper layers, 254.9 x 62.2 mm, 93 parts, among them K1 KEYSW, K10 KEYSW, K11 KEYSW, K12 KEYSW, K14 KEYSW, K15 KEYSW, K16 KEYSW, K17 KEYSW, K18 KEYSW, K19 KEYSW, K2 KEYSW, K20 KEYSW, K21 KEYSW, K22 KEYSW, K23 KEYSW, K24 KEYSW, K25 KEYSW, K27 KEYSW, K28 KEYSW, K29 KEYSW, K3 KEYSW, K30 KEYSW, K31 KEYSW, K32 KEYSW, K33 KEYSW, K34 KEYSW, K35 KEYSW, K36 KEYSW, K37 KEYSW, K4 KEYSW, K5 KEYSW, K6 KEYSW, K7 KEYSW, K8 KEYSW, K9 KEYSW, M2_1 VAL**, M2_2 VAL**, M2_3 VAL**, M2_4 VAL**, M2_5 VAL**, M2_6 VAL**, M2_7 VAL**, SW2 SW_SPDT

Commit message: Push graphics and gerbers of V1.1
Parts:
- moved M2_6 19.1 mm to (243.0, 95.1)
- moved M2_7 13.2 mm to (283.3, 76.0)
Routing:
- net RowD: track 317.1 -> 320.5 mm
Changed lines of the file:
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@@
     (thickness 1.6)
     (drawings 22)
-    (tracks 1327)
+    (tracks 1328)
     (zones 0)
     (modules 93)
@@
       (padsonsilk false)
       (subtractmaskfromsilk false)
-      (outputformat 5)
+      (outputformat 1)
       (mirror false)
       (drillshape 0)
       (scaleselection 1)
-      (outputdirectory "svg/"))
+      (outputdirectory "gerber/"))
   )
   (net 0 "")
@@
   )
   (module kbd:spacer_m2 (layer F.Cu)
-    (at 242.9 76.03)
+    (at 243.006 95.146)
     (descr "Mounting Hole 2.2mm, no annular, M2")
     (tags "mounting hole 2.2mm no annular m2")
@@
     (pad "" np_thru_hole circle (at 0 0) (size 4.3 4.3) (drill 4.3) (layers *.Cu *.Mask))
   )
-  (module kbd:spacer_m2 (layer F.Cu)
-    (at 296.51 77.42)
+  (module kbd:spacer_m2 locked (layer F.Cu)
+    (at 283.336 76.036)
     (descr "Mounting Hole 2.2mm, no annular, M2")
     (tags "mounting hole 2.2mm no annular m2")
@@
   (segment (start 185.74 106.8795) (end 185.74 107.442) (width 0.25) (layer B.Cu) (net 39))
   (segment (start 185.74 106.8795) (end 185.74 106.317) (width 0.25) (layer B.Cu) (net 39))
-  (segment (start 72.8 108.2) (end 73.9253 108.2) (width 0.25) (layer F.Cu) (net 39))
-  (segment (start 127.3 108.5) (end 126.1747 108.5) (width 0.25) (layer F.Cu) (net 39))
-  (segment (start 126.1747 108.5) (end 124.7702 109.9045) (width 0.25) (layer F.Cu) (net 39))
-  (segment (start 124.7702 109.9045) (end 75.3485 109.9045) (width 0.25) (layer F.Cu) (net 39))
-  (segment (start 75.3485 109.9045) (end 73.9253 108.4813) (width 0.25) (layer F.Cu) (net 39))
-  (segment (start 73.9253 108.4813) (end 73.9253 108.2) (width 0.25) (layer F.Cu) (net 39))
   (segment (start 129.8 108.5) (end 127.3 108.5) (width 0.25) (layer F.Cu) (net 39))
   (segment (start 72.8 105.875) (end 72.8 104.9497) (width 0.25) (layer B.Cu) (net 39))
@@
   (segment (start 243.078 108.04) (end 243.078 106.84) (width 0.25) (layer B.Cu) (net 39))
   (segment (start 243.078 106.84) (end 243.078 105.715) (width 0.25) (layer B.Cu) (net 39))
+  (segment (start 73.4545 109.9045) (end 72.8 109.25) (width 0.25) (layer F.Cu) (net 39))
+  (segment (start 124.7702 109.9045) (end 73.4545 109.9045) (width 0.25) (layer F.Cu) (net 39))
+  (segment (start 126.1747 108.5) (end 124.7702 109.9045) (width 0.25) (layer F.Cu) (net 39))
+  (segment (start 72.8 109.25) (end 72.8 108.2) (width 0.25) (layer F.Cu) (net 39))
+  (segment (start 127.3 108.5) (end 126.1747 108.5) (width 0.25) (layer F.Cu) (net 39))
   (segment (start 66.699 63.0885) (end 66.9125 62.875) (width 0.25) (layer B.Cu) (net 40))
   (segment (start 65.7377 80.645) (end 65.792 80.5907) (width 0.25) (layer B.Cu) (net 40))
@@
   (segment (start 283.464 86.157) (end 283.464 85.2317) (width 0.25) (layer B.Cu) (net 57))
   (segment (start 283.464 85.2317) (end 282.3387 84.1064) (width 0.25) (layer B.Cu) (net 57))
-  (segment (start 282.3387 84.1064) (end 282.3387 72.4956) (width 0.25) (layer B.Cu) (net 57))
-  (segment (start 282.3387 72.4956) (end 283.464 71.3703) (width 0.25) (layer B.Cu) (net 57))
-  (segment (start 283.464 70.245) (end 283.464 71.3703) (width 0.25) (layer B.Cu) (net 57))
   (segment (start 283.566 106.231) (end 283.566 107.356) (width 0.25) (layer B.Cu) (net 57))
   (segment (start 262.276 107.176) (end 262.276 108.376) (width 0.25) (layer B.Cu) (net 57))
@@
   (segment (start 239.916 74.4813) (end 239.916 82.0187) (width 0.25) (layer B.Cu) (net 57))
   (segment (start 242.824 70.448) (end 242.824 71.5733) (width 0.25) (layer B.Cu) (net 57))
+  (segment (start 282.3387 84.1064) (end 282.3387 81.7887) (width 0.25) (layer B.Cu) (net 57))
+  (segment (start 282.3387 81.7887) (end 278.966 78.416) (width 0.25) (layer B.Cu) (net 57))
+  (segment (start 282.414 70.245) (end 283.464 70.245) (width 0.25) (layer B.Cu) (net 57))
+  (segment (start 278.966 73.693) (end 282.414 70.245) (width 0.25) (layer B.Cu) (net 57))
+  (segment (start 278.966 78.416) (end 278.966 73.693) (width 0.25) (layer B.Cu) (net 57))
   (segment (start 302.2 97.75) (end 302.0996 99.2235) (width 0.25) (layer F.Cu) (net 58))
   (segment (start 302.0996 99.2235) (end 302.0996 99.6504) (width 0.25) (layer F.Cu) (net 58))
