File: PRKL30.sch (KiCad schematic (older format))
At the start: 83 parts, among them K1 KEYSW, K10 KEYSW, K11 KEYSW, K12 KEYSW, K14 KEYSW, K15 KEYSW, K16 KEYSW, K17 KEYSW, K18 KEYSW, K19 KEYSW, K2 KEYSW, K20 KEYSW, K21 KEYSW, K22 KEYSW, K23 KEYSW, K24 KEYSW, K25 KEYSW, K27 KEYSW, K28 KEYSW, K29 KEYSW, K3 KEYSW, K30 KEYSW, K31 KEYSW, K32 KEYSW, K33 KEYSW, K34 KEYSW, K35 KEYSW, K36 KEYSW, K37 KEYSW, K4 KEYSW, K5 KEYSW, K6 KEYSW, K7 KEYSW, K8 KEYSW, K9 KEYSW

Commit message: Change project name, clean up older files
Parts:
- added Feather1: Adafruit32u4BLE, SpaceLib:Adafruit32u4BLE, symbol PRKL30-rescue:Adafruit32u4BLE-Spacelib-Memekeeb-feather-rescue
- added SW2: SW_SPDT, Button_Switch_SMD:SW_SPDT_PCM12, symbol Switch:SW_SPDT
- D1, D10, D11, D12, D13, D14, D15, D16, D17, D18, D19, D2, D20, D21, D22, D23, D24, D25, D27, D28, D29, D3, D30, D31, D32, D33, D34, D35, D36, D37, D4, D5, D6, D7, D8, D9, D_1.25u1, D_ISOENTR1: symbol keyboard_parts:D -> PRKL30-rescue:D-keyboard_parts-Memekeeb-rescue-Memekeeb-feather-rescue
- K1, K10, K11, K12, K14, K15, K16, K17, K18, K19, K2, K20, K21, K22, K23, K24, K25, K27, K28, K29, K3, K30, K31, K32, K33, K34, K35, K36, K37, K4, K5, K6, K7, K8, K9, K_1.25u1, K_2Uspc1, K_BCKSPC1, K_ISOENTER1: symbol keyboard_parts:KEYSW -> PRKL30-rescue:KEYSW-keyboard_parts-Memekeeb-rescue-Memekeeb-feather-rescue
- MCU_Pro_Micr0: symbol keebio:ProMicro -> PRKL30-rescue:ProMicro-keebio-Memekeeb-rescue-Memekeeb-feather-rescue
- SW_RST1: symbol keyboard_parts:SW_PUSH -> PRKL30-rescue:SW_PUSH-keyboard_parts-Memekeeb-rescue-Memekeeb-feather-rescue
Connections:
- net ColA: now also Feather1.27 (TX)
- net ColB: now also Feather1.12 (SDA)
- net ColC: now also Feather1.6 (11)
- net ColD: now also Feather1.5 (12)
- net ColE: now also Feather1.4 (13)
- net ColF: now also Feather1.7 (10)
- net ColG: now also Feather1.8 (9)
- net ColH: now also Feather1.9 (6)
- net ColI: now also Feather1.10 (5)
- net ColJ: now also Feather1.11 (SCL)
- net EncA: now also Feather1.17 (A0)
- net EncB: now also Feather1.18 (A1)
- net GND: now also Feather1.16 (GND), SW2.2 (B)
- net RGB: now also Feather1.19 (A2)
- net RGB_PWR: now also MCU_Pro_Micr0.24 (RAW), Feather1.3 (USB); no longer MCU_Pro_Micr0.21 (VCC)
- net RST: now also Feather1.13 (Reset)
- net RowA: now also Feather1.20 (A3)
- net RowB: now also Feather1.21 (A4)
- net RowC: now also Feather1.22 (A5)
- net RowD: now also Feather1.26 (RX)
- new net DP1: Feather1.2 (En), SW2.1 (A)
- no-connect marks 4 -> 12
Other:
- moved on the sheet: MCU_Pro_Micr0
